File: rev1/pcb/om.kicad_pcb (KiCad board)
At the start: 2 copper layers, 124.4 x 111.4 mm, 19 parts

Commit message: Updated Om silkscreens to look more dynamic
Other:
- outline, holes or cut-outs redrawn
- board text added: "PROBLEM"
- board text added: "PROGRAM"
- board text added: "SUFFERING"
- board text added: "TOO BUSY"
- board text added: "TRAINING"
- board text added: "UNWORTHINESS"
- board text added: "WISE"
- board text added: "Your"
- board text added: "for becoming"
- board text added: "holding on to your"
- board text added: "is part of our"
- board text added: "is you are"
Changed lines of the file:
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@@
   (gr_arc (start 119.4 105.1) (mid 169.415908 79.055538) (end 224.45 91.35) (layer "Edge.Cuts") (width 0.2))
   (gr_line (start 190.4 169.2) (end 227.25 189.75) (layer "Edge.Cuts") (width 0.2))
-  (gr_line (start 124.45 160.85) (end 190.4 169.2) (layer "Edge.Cuts") (width 0.2))
+  (gr_line (start 124.4 160.75) (end 190.4 169.2) (layer "Edge.Cuts") (width 0.2))
   (gr_line (start 243.8 91.35) (end 224.45 91.35) (layer "Edge.Cuts") (width 0.2))
+  (gr_text "TOO BUSY" (at 229 153) (layer "F.Cu")
+    (effects (font (size 3 3) (thickness 0.3)))
+  )
+  (gr_text "PROBLEM" (at 230 149) (layer "F.Cu")
+    (effects (font (size 3 3) (thickness 0.3)))
+  )
+  (gr_text "UNWORTHINESS" (at 232 157) (layer "F.Cu")
+    (effects (font (size 3 1.9) (thickness 0.3)))
+  )
+  (gr_text "WISE" (at 223 159) (layer "B.Cu")
+    (effects (font (size 3 5) (thickness 0.3)) (justify mirror))
+  )
+  (gr_text "SUFFERING" (at 231 147) (layer "B.Cu")
+    (effects (font (size 3 3) (thickness 0.3)) (justify mirror))
+  )
+  (gr_text "PROGRAM" (at 227 154) (layer "B.Cu")
+    (effects (font (size 1.5 4.8) (thickness 0.3)) (justify mirror))
+  )
+  (gr_text "TRAINING" (at 227 151) (layer "B.Cu")
+    (effects (font (size 2.5 5) (thickness 0.3)) (justify mirror))
+  )
+  (gr_text "SUFFERING" (at 231 147) (layer "B.Paste")
+    (effects (font (size 3 3) (thickness 0.3)) (justify mirror))
+  )
+  (gr_text "WISE" (at 223 159) (layer "B.Paste")
+    (effects (font (size 3 5) (thickness 0.3)) (justify mirror))
+  )
+  (gr_text "PROGRAM" (at 227 154) (layer "B.Paste")
+    (effects (font (size 1.5 4.8) (thickness 0.3)) (justify mirror))
+  )
+  (gr_text "TRAINING" (at 227 151) (layer "B.Paste")
+    (effects (font (size 2.5 5) (thickness 0.3)) (justify mirror))
+  )
+  (gr_text "PROBLEM" (at 230 149) (layer "F.Paste")
+    (effects (font (size 3 3) (thickness 0.3)))
+  )
+  (gr_text "TOO BUSY" (at 229 153) (layer "F.Paste")
+    (effects (font (size 3 3) (thickness 0.3)))
+  )
+  (gr_text "UNWORTHINESS" (at 232 157) (layer "F.Paste")
+    (effects (font (size 3 1.9) (thickness 0.3)))
+  )
+  (gr_text "for \nbecoming" (at 243 158) (layer "B.SilkS")
+    (effects (font (size 1.5 1.5) (thickness 0.25)) (justify left mirror))
+  )
+  (gr_text "is part\nof our" (at 214 147) (layer "B.SilkS")
+    (effects (font (size 1.5 1.5) (thickness 0.3)) (justify mirror))
+  )
+  (gr_text "holding on\nto your" (at 216 157) (layer "F.SilkS")
+    (effects (font (size 1 1) (thickness 0.25)))
+  )
+  (gr_text "is you\nare" (at 215 153) (layer "F.SilkS")
+    (effects (font (size 1 1) (thickness 0.25)))
+  )
+  (gr_text "Your" (at 216.700981 148.860693) (layer "F.SilkS")
+    (effects (font (size 1.5 1.3) (thickness 0.3)))
+  )
   (segment (start 241.27 118.772868) (end 219.993828 140.04904) (width 0.25) (layer "F.Cu") (net 2))
   (segment (start 241.27 118.04) (end 241.27 118.772868) (width 0.25) (layer "F.Cu") (net 2))

Commit message: Added gerbers
Routing:
- net P16: track 55.1 -> 57.5 mm
- net P18: track 84.6 -> 86.7 mm
- net P14: track 43.3 -> 44.4 mm
- net P19: track 55.9 -> 56.8 mm
