File: rev3/pcb/om.kicad_pcb (KiCad board)
At the start: 2 copper layers, 128.3 x 108.8 mm, 49 parts, among them J1 USB_C_Receptacle, J2 JST-BATT, J3 USB, J4 SWD, J5 USB, Q1 AO3407, Q2 AO3407, SW1 Choc, SW10 Choc, SW11 Choc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

Commit message: Fix the USB port connections, time to start routing
Parts:
- moved J4 6.71 mm to (292.2, 126.5), turned to 90 degrees
- moved J5 6.00 mm to (292.2, 123.5), turned to 90 degrees
- moved U1 5.10 mm to (296.2, 125.5), turned to -90 degrees
- moved J1 1.07 mm to (296.2, 66.5)
- turned R2 to -90 degrees

Commit message: Fix up the schematic -> footprint library usage.  Pins were on the wrong pads.
Parts:
- removed ? (x2): , 
- removed J3: USB, Connector_PinHeader_2.00mm:PinHeader_1x04_P2.00mm_Vertical
- removed J5: USB, Connector_PinSocket_2.00mm:PinSocket_1x04_P2.00mm_Vertical
- removed _1: Tenting Puck, Tenting Puck
- moved R7 7.52 mm to (298.9, 96.1), turned to -45 degrees
- moved C1 5.71 mm to (289.2, 93.2)
- moved C2 5.71 mm to (286.2, 102.2)
- moved D1 5.71 mm to (298.2, 91.2)
- moved D2 5.71 mm to (296.1, 91.2)
- moved D3 5.71 mm to (286.2, 94.2)
- moved ESD1 5.71 mm to (287.2, 87.2)
- moved Q1 5.71 mm to (286.2, 91.2)
- moved Q2 5.71 mm to (293.2, 93.2)
- moved R1 5.71 mm to (297.2, 83.2)
- moved R2 5.71 mm to (293.2, 83.2)
- moved R3 5.71 mm to (287.2, 107.0)
- moved R4 5.71 mm to (291.1, 97.2), turned to -90 degrees
- moved R5 5.71 mm to (295.2, 97.2)
- moved R8 5.71 mm to (300.2, 93.2)
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Connections:
- U1 pad 14: +3V3 -> unconnected-(U1-Pad14)
- U1 pad 15: /unconnected-(U1-P0.07) -> unconnected-(U1-Pad15)
- U1 pad 16: BLUE_LED -> unconnected-(U1-Pad16)
- U1 pad 17: /unconnected-(U1-P0.12) -> unconnected-(U1-Pad17)
- U1 pad 18: SCL -> unconnected-(U1-Pad18)
- U1 pad 19: SDA -> unconnected-(U1-Pad19)
- U1 pad 20: /unconnected-(U1-P0.19) -> unconnected-(U1-Pad20)
- U1 pad 21: RESET -> unconnected-(U1-Pad21)
- U1 pad 22: VBUS -> unconnected-(U1-Pad22)
- U1 pad 23: D- -> unconnected-(U1-Pad23)
- U1 pad 24: D+ -> unconnected-(U1-Pad24)
- U1 pad 25: GND -> unconnected-(U1-Pad25)
- U1 pad 26: SW10 -> unconnected-(U1-Pad26)
- U1 pad 27: SW9 -> unconnected-(U1-Pad27)
- U1 pad 28: SW8 -> unconnected-(U1-Pad28)
- U1 pad 29: SW7 -> unconnected-(U1-Pad29)
- U1 pad 30: SW15 -> unconnected-(U1-Pad30)
- U1 pad 31: SWDCLK -> unconnected-(U1-Pad31)
- U1 pad 32: SWDIO -> GND
- U1 pad 33: SW14 -> SW11
- U1 pad 34: SW13 -> SW6
- U1 pad 35: SW6 -> SW13
- U1 pad 36: SW11 -> SW14
- U1 pad 37: GND -> SWDIO
- U1 pad 38: unconnected-(U1-Pad38) -> SWDCLK
- U1 pad 39: unconnected-(U1-Pad39) -> SW15
- U1 pad 40: unconnected-(U1-Pad40) -> SW7
- U1 pad 41: unconnected-(U1-Pad41) -> SW8
- U1 pad 42: unconnected-(U1-Pad42) -> SW9
- U1 pad 43: unconnected-(U1-Pad43) -> SW10
- U1 pad 44: unconnected-(U1-Pad44) -> GND
- U1 pad 45: unconnected-(U1-Pad45) -> D+
- U1 pad 46: unconnected-(U1-Pad46) -> D-
- U1 pad 47: unconnected-(U1-Pad47) -> VBUS
- U1 pad 48: unconnected-(U1-Pad48) -> RESET
- U1 pad 49: unconnected-(U1-Pad49) -> /unconnected-(U1-P0.19)
- U1 pad 50: unconnected-(U1-Pad50) -> SDA
- U1 pad 51: unconnected-(U1-Pad51) -> SCL
- U1 pad 52: unconnected-(U1-Pad52) -> /unconnected-(U1-P0.12)
- U1 pad 53: unconnected-(U1-Pad53) -> BLUE_LED
- U1 pad 54: unconnected-(U1-Pad54) -> /unconnected-(U1-P0.07)
- U1 pad 55: unconnected-(U1-Pad55) -> +3V3
Routing:
- net VBUS: track 0.00 -> 90.4 mm, vias 0 -> 9
- net D-: track 0.00 -> 59.2 mm, vias 0 -> 1
- net D+: track 0.00 -> 55.9 mm, vias 0 -> 2
- net +BATT: track 0.00 -> 54.8 mm, vias 0 -> 2
- net +3V3: track 0.00 -> 48.6 mm, vias 0 -> 1
- net Earth: track 0.00 -> 41.6 mm, vias 0 -> 2
- net BLUE_LED: track 0.00 -> 40.4 mm, vias 0 -> 2
- net VCC_CONTROL: track 0.00 -> 32.0 mm, vias 0 -> 3
- net /BAT+_SWITCHED: track 0.00 -> 30.8 mm, vias 0 -> 6
- net VSENSE: track 0.00 -> 30.1 mm
- net /Net-(U3-PROG): track 0.00 -> 28.7 mm, vias 0 -> 2
- net USBD+: track 0.00 -> 27.4 mm, vias 0 -> 3
- net USBD-: track 0.00 -> 27.0 mm, vias 0 -> 2
- net Net-(J1-PadA5): track 0.00 -> 25.5 mm, vias 0 -> 2
- net Net-(J1-PadB5): track 0.00 -> 24.1 mm, vias 0 -> 2
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
Commit message: Routing might be done?
Parts:
- added J2: JST-BATT, Connector_JST:JST_PH_S2B-PH-K_1x02_P2.00mm_Horizontal, B.Cu at (243.6, 161.1)
- R_TACT1: footprint Button_Switch_SMD:SW_SPST_TL3342 -> om-footprints:SKHLLCA010
- SW1, SW10, SW11, SW12, SW13, SW14, SW15, SW16, SW17, SW2, SW3, SW4, SW5, SW6, SW7, SW8, SW9: footprint kleeb-pg1350:pg1350-R -> kleeb-pg1350:pg1350-DR
- moved SW_POW1 61.6 mm to (264.0, 162.0)
- moved R5 52.9 mm to (256.3, 133.1), turned to -90 degrees
- moved C1 52.4 mm to (251.4, 129.5), turned to -90 degrees
- moved R2 51.6 mm to (248.8, 109.7), turned to 0 degrees
- moved R9 51.4 mm to (254.3, 123.7), turned to 0 degrees
- moved D3 50.9 mm to (248.9, 128.8)
- moved SW5 50.9 mm to (177.0, 124.1)
- moved SW15 50.9 mm to (236.9, 145.1)
- moved SW10 50.9 mm to (218.9, 108.1)
- moved SW6 50.9 mm to (177.0, 141.1)
- moved Q1 50.9 mm to (248.9, 125.8)
- moved SW4 50.9 mm to (177.0, 107.1)
- moved U3 50.9 mm to (265.9, 127.8)
- moved C2 50.9 mm to (248.9, 136.8)
- moved SW17 50.9 mm to (246.9, 186.2)
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Connections:
- SW1 pad 1: SW1 -> Col1
- SW1 pad 2: GND -> Row1
- SW10 pad 1: SW4 -> Col4
- SW10 pad 2: GND -> Row1
- SW11 pad 1: SW9 -> Col4
- SW11 pad 2: GND -> Row2
- SW12 pad 1: SW14 -> Col4
- SW12 pad 2: GND -> Row3
- SW13 pad 1: SW5 -> Col5
- SW13 pad 2: GND -> Row1
- SW14 pad 1: SW10 -> Col5
- SW14 pad 2: GND -> Row2
- SW15 pad 1: SW15 -> Col5
- SW15 pad 2: GND -> Row3
- SW16 pad 1: SW16 -> Col4
- SW16 pad 2: GND -> Row4
- SW17 pad 1: SW17 -> Col5
- SW17 pad 2: GND -> Row4
- SW2 pad 1: SW6 -> Col1
- SW2 pad 2: GND -> Row2
- SW3 pad 1: SW11 -> Col1
- SW3 pad 2: GND -> Row3
- SW4 pad 1: SW2 -> Col2
- SW4 pad 2: GND -> Row1
- SW5 pad 1: SW7 -> Col2
- SW5 pad 2: GND -> Row2
- SW6 pad 1: SW12 -> Col2
- SW6 pad 2: GND -> Row3
- SW7 pad 1: SW3 -> Col3
- SW7 pad 2: GND -> Row1
- SW8 pad 1: SW8 -> Col3
- SW8 pad 2: GND -> Row2
- SW9 pad 1: SW13 -> Col3
- SW9 pad 2: GND -> Row3
- U1 pad 10: SW4 -> unconnected-(U1-Pad10)
- U1 pad 13: SW5 -> unconnected-(U1-Pad13)
- U1 pad 2: SW17 -> Col1
- U1 pad 3: SW16 -> Col2
- U1 pad 33: SW11 -> unconnected-(U1-Pad33)
- U1 pad 34: SW6 -> unconnected-(U1-Pad34)
- U1 pad 35: SW13 -> Row4
- U1 pad 36: SW14 -> Row3
- U1 pad 39: SW15 -> Row2
- U1 pad 4: SW1 -> Col3
- U1 pad 40: SW7 -> Row1
- U1 pad 41: SW8 -> Col5
- U1 pad 42: SW9 -> unconnected-(U1-Pad42)
- U1 pad 43: SW10 -> unconnected-(U1-Pad43)
- U1 pad 49: /unconnected-(U1-P0.19) -> unconnected-(U1-Pad49)
- U1 pad 5: SW12 -> Col4
- U1 pad 52: /unconnected-(U1-P0.12) -> unconnected-(U1-Pad52)
- U1 pad 54: /unconnected-(U1-P0.07) -> unconnected-(U1-Pad54)
- U1 pad 8: SW2 -> unconnected-(U1-Pad8)
- U1 pad 9: SW3 -> unconnected-(U1-Pad9)
Routing:
- net (no net): track 0.00 -> 372.8 mm, vias 0 -> 17
- net Col1: track 0.00 -> 203.5 mm, vias 0 -> 3
- net Col2: track 0.00 -> 201.1 mm, vias 0 -> 3
- net Col3: track 0.00 -> 183.1 mm, vias 0 -> 3
- net Row1: track 0.00 -> 172.7 mm, vias 0 -> 5
- net Col4: track 0.00 -> 165.8 mm, vias 0 -> 3
- net Row2: track 0.00 -> 155.3 mm, vias 0 -> 5
- net Row3: track 0.00 -> 141.2 mm, vias 0 -> 5
- net Col5: track 0.00 -> 137.7 mm, vias 0 -> 1
- net GND: track 3.94 -> 84.0 mm, vias 15 -> 10
- net Row4: track 0.00 -> 79.5 mm, vias 0 -> 4
- net RESET: track 0.00 -> 31.5 mm, vias 0 -> 2
- net D-: track 59.2 -> 38.2 mm, vias 1 -> 2
- net D+: track 55.9 -> 35.5 mm
- net /BAT+_SWITCHED: track 30.8 -> 50.1 mm
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Other:
- outline, holes or cut-outs redrawn

Commit message: Mostly in place, time to refactor
Parts:
- added DIODE1: 1N914WT, Diode_SMD:D_SOD-123, F.Cu at (150.3, 129.9)
- added DIODE10: 1N914WT, Diode_SMD:D_SOD-123, F.Cu at (217.7, 129.8)
- added DIODE11: 1N914WT, Diode_SMD:D_SOD-123, F.Cu at (217.7, 112.8)
- added DIODE12: 1N914WT, Diode_SMD:D_SOD-123, F.Cu at (217.7, 146.8)
- added DIODE13: 1N914WT, Diode_SMD:D_SOD-123, F.Cu at (235.7, 115.8)
- added DIODE14: 1N914WT, Diode_SMD:D_SOD-123, F.Cu at (235.7, 132.8)
- added DIODE15: 1N914WT, Diode_SMD:D_SOD-123, F.Cu at (235.7, 149.8)
- added DIODE16: 1N914WT, Diode_SMD:D_SOD-123, F.Cu at (226.3, 182.4)
- added DIODE17: 1N914WT, Diode_SMD:D_SOD-123, F.Cu at (243.4, 190.3)
- added DIODE2: 1N914WT, Diode_SMD:D_SOD-123, F.Cu at (151.8, 146.8)
- added DIODE3: 1N914WT, Diode_SMD:D_SOD-123, F.Cu at (153.2, 163.8)
- added DIODE4: 1N914WT, Diode_SMD:D_SOD-123, F.Cu at (175.8, 111.8)
- added DIODE5: 1N914WT, Diode_SMD:D_SOD-123, F.Cu at (175.8, 128.8)
- added DIODE6: 1N914WT, Diode_SMD:D_SOD-123, F.Cu at (175.8, 145.8)
- added DIODE7: 1N914WT, Diode_SMD:D_SOD-123, F.Cu at (198.7, 104.8)
- added DIODE8: 1N914WT, Diode_SMD:D_SOD-123, F.Cu at (198.7, 121.8)
- added DIODE9: 1N914WT, Diode_SMD:D_SOD-123, F.Cu at (198.7, 138.8)
- SW1, SW10, SW11, SW12, SW13, SW14, SW15, SW16, SW17, SW2, SW3, SW4, SW5, SW6, SW7, SW8, SW9: footprint kleeb-pg1350:pg1350-DR -> kleeb-pg1350:pg1350
- moved D3 6.28 mm to (253.9, 125.0), turned to 0 degrees
- moved C1 3.07 mm to (248.5, 128.6), turned to 0 degrees
- moved R9 1.78 mm to (252.7, 123.0)
- moved D2 1.17 mm to (257.6, 125.9)
- moved SW8 1.17 mm to (198.7, 117.1)
- moved R10 1.17 mm to (247.7, 107.4)
- moved SW3 1.17 mm to (152.8, 159.1)
- moved U3 1.17 mm to (264.7, 127.8)
- moved R4 1.17 mm to (253.4, 114.5)
- moved R5 1.17 mm to (255.2, 133.2)
- moved SW17 1.17 mm to (245.8, 186.2)
- moved R_TACT1 1.17 mm to (257.9, 176.0)
- moved C3 1.17 mm to (247.9, 103.2)
- moved SW13 1.17 mm to (235.7, 111.1)
- moved J4 1.17 mm to (253.6, 148.1)
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- renumbered J2 to J3
Connections:
- R7 pad 2: GND -> VSENSE_ENABLE
- SW1 pad 2: Row1 -> Net-(DIODE1-Pad2)
- SW10 pad 2: Row1 -> Net-(DIODE10-Pad2)
- SW11 pad 2: Row2 -> Net-(SW11-Pad2)
- SW12 pad 2: Row3 -> Net-(DIODE12-Pad2)
- SW13 pad 2: Row1 -> Net-(SW13-Pad2)
- SW14 pad 2: Row2 -> Net-(SW14-Pad2)
- SW15 pad 2: Row3 -> Net-(SW15-Pad2)
- SW16 pad 2: Row4 -> Net-(SW16-Pad2)
- SW17 pad 2: Row4 -> Net-(SW17-Pad2)
- SW2 pad 2: Row2 -> Net-(SW2-Pad2)
- SW3 pad 2: Row3 -> Net-(DIODE3-Pad2)
- SW4 pad 2: Row1 -> Net-(DIODE4-Pad2)
- SW5 pad 2: Row2 -> Net-(DIODE5-Pad2)
- SW6 pad 2: Row3 -> Net-(DIODE6-Pad2)
- SW7 pad 2: Row1 -> Net-(DIODE7-Pad2)
- SW8 pad 2: Row2 -> Net-(DIODE8-Pad2)
- SW9 pad 2: Row3 -> Net-(DIODE9-Pad2)
- U1 pad 10: unconnected-(U1-Pad10) -> VSENSE_ENABLE
- U1 pad 6: P0.03 -> unconnected-(U1-Pad6)
- U1 pad 7: P0.02 -> unconnected-(U1-Pad7)
Routing:
- net (no net): track 372.8 -> 0.00 mm, vias 17 -> 0
- net Net-(DIODE10-Pad2): track 0.00 -> 19.4 mm
- net VSENSE_ENABLE: track 0.00 -> 15.8 mm, vias 0 -> 2
- net Row2: track 155.3 -> 142.9 mm, vias 5 -> 0
- net Row3: track 141.2 -> 128.9 mm, vias 5 -> 0
- net Row1: track 172.7 -> 160.4 mm, vias 5 -> 0
- net Col1: track 203.5 -> 215.6 mm
- net Net-(DIODE1-Pad2): track 0.00 -> 9.69 mm
- net Net-(SW14-Pad2): track 0.00 -> 9.69 mm
- net Net-(DIODE8-Pad2): track 0.00 -> 9.69 mm
- net Net-(SW13-Pad2): track 0.00 -> 9.69 mm
- net Net-(DIODE7-Pad2): track 0.00 -> 9.69 mm
- net Net-(DIODE6-Pad2): track 0.00 -> 9.69 mm
- net Net-(DIODE5-Pad2): track 0.00 -> 9.69 mm
- net Net-(DIODE12-Pad2): track 0.00 -> 9.69 mm
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